File: _autosave-leddings.kicad_pcb (KiCad board)
At the start: 2 copper layers, 50.8 x 82.6 mm, 39 parts, among them J4 Conn_01x04, J5 Micro USB, J6 Barrel_Jack, J7 Conn_01x04, J8 Conn_01x04, Q1 IRLR8726TRLPBF, Q2 IRLR8726TRLPBF, Q3 IRLR8726TRLPBF, SW1 SW_RESET, SW2 Boot SEL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

Commit message: changed some parts to smd, fixed some design errors
Other:
- board text added: "Alexander Schramm Wifi RGB Driver Oct 2018 v1.1"
- board text removed: "Alexander Schramm Wifi RGB Driver Oct 2018 v1.0"
Changed lines of the file:
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@@
     (34 B.Paste user)
     (35 F.Paste user)
-    (36 B.SilkS user hide)
+    (36 B.SilkS user)
     (37 F.SilkS user)
     (38 B.Mask user)
@@
     (visible_elements FFFFEF7F)
     (pcbplotparams
-      (layerselection 0x010fc_ffffffff)
-      (usegerberextensions false)
-      (usegerberattributes false)
+      (layerselection 0x010f0_ffffffff)
+      (usegerberextensions true)
+      (usegerberattributes true)
       (usegerberadvancedattributes false)
-      (creategerberjobfile false)
+      (creategerberjobfile true)
       (excludeedgelayer true)
-      (linewidth 0.100000)
+      (linewidth 0.150000)
       (plotframeref false)
       (viasonmask false)
       (mode 1)
-      (useauxorigin false)
+      (useauxorigin true)
       (hpglpennumber 1)
       (hpglpenspeed 20)
@@
     (effects (font (size 1 1) (thickness 0.2)) (justify right))
   )
-  (gr_text "Alexander Schramm\nWifi RGB Driver\nOct 2018\nv1.0" (at 152.908 69.85) (layer B.SilkS)
+  (gr_text "Alexander Schramm\nWifi RGB Driver\nOct 2018\nv1.1" (at 152.908 69.85) (layer B.SilkS)
     (effects (font (size 1.5 1.5) (thickness 0.3)) (justify mirror))
   )
