File: _saved_smarts.sch (KiCad schematic (older format))
At the start: 6 parts, among them SW1 SW_RESET, SW2 Boot SEL, U3 ESP-12E

Commit message: changed some parts to smd, fixed some design errors
Parts:
- C6: footprint (none) -> Resistor_SMD:R_0805_2012Metric_Pad1.15x1.40mm_HandSolder
Changed lines of the file:
@@
 F 0 "C6" H 4115 4846 50  0000 L CNN
 F 1 "10uF" H 4115 4755 50  0000 L CNN
-F 2 "" H 4038 4650 50  0001 C CNN
+F 2 "Resistor_SMD:R_0805_2012Metric_Pad1.15x1.40mm_HandSolder" H 4038 4650 50  0001 C CNN
 F 3 "~" H 4000 4800 50  0001 C CNN
 	1    4000 4800
