File: driver.sch (KiCad schematic (older format))
At the start: 10 parts

Commit message: added stuff
Parts:
- J2: renamed from J?; footprint (none) -> Pin_Headers:Pin_Header_Straight_1x04_Pitch2.54mm
- Q1, Q2, Q3: renamed from Q?; footprint (none) -> TO_SOT_Packages_THT:TO-220-3_Vertical
- R1, R2, R3, R4, R5, R6: renamed from R?; footprint (none) -> Resistors_SMD:R_0805_HandSoldering
Changed lines of the file:
@@
 $EndDescr
 $Comp
-L Q_NMOS_GDS Q?
+L Q_NMOS_GDS Q1
 U 1 1 5B157B68
 P 3600 2000
-F 0 "Q?" H 3800 2050 50  0000 L CNN
+F 0 "Q1" H 3800 2050 50  0000 L CNN
 F 1 "FQP30N06L" H 3800 1950 50  0000 L CNN
-F 2 "" H 3800 2100 50  0001 C CNN
+F 2 "TO_SOT_Packages_THT:TO-220-3_Vertical" H 3800 2100 50  0001 C CNN
 F 3 "" H 3600 2000 50  0001 C CNN
 	1    3600 2000
@@
 $EndComp
 $Comp
-L R R?
+L R R1
 U 1 1 5B157EE6
 P 2900 2000
-F 0 "R?" V 2980 2000 50  0000 C CNN
+F 0 "R1" V 2980 2000 50  0000 C CNN
 F 1 "100R" V 2900 2000 50  0000 C CNN
-F 2 "" V 2830 2000 50  0001 C CNN
+F 2 "Resistors_SMD:R_0805_HandSoldering" V 2830 2000 50  0001 C CNN
 F 3 "" H 2900 2000 50  0001 C CNN
 	1    2900 2000
@@
 $EndComp
 $Comp
-L R R?
+L R R4
 U 1 1 5B157F0E
 P 3200 2300
-F 0 "R?" V 3280 2300 50  0000 C CNN
+F 0 "R4" V 3280 2300 50  0000 C CNN
 F 1 "10K" V 3200 2300 50  0000 C CNN
-F 2 "" V 3130 2300 50  0001 C CNN
+F 2 "Resistors_SMD:R_0805_HandSoldering" V 3130 2300 50  0001 C CNN
 F 3 "" H 3200 2300 50  0001 C CNN
 	1    3200 2300
@@
 	7050 3700 7400 3700
 $Comp
-L Conn_01x04 J?
+L Conn_01x04 J2
 U 1 1 5B158040
 P 7600 3600
-F 0 "J?" H 7600 3800 50  0000 C CNN
+F 0 "J2" H 7600 3800 50  0000 C CNN
 F 1 "Conn_01x04" H 7600 3300 50  0000 C CNN
-F 2 "" H 7600 3600 50  0001 C CNN
+F 2 "Pin_Headers:Pin_Header_Straight_1x04_Pitch2.54mm" H 7600 3600 50  0001 C CNN
 F 3 "" H 7600 3600 50  0001 C CNN
 	1    7600 3600
@@
 $EndComp
 $Comp
-L +12V #PWR013
+L +12V #PWR07
 U 1 1 5B1580E3
 P 7050 3800
-F 0 "#PWR013" H 7050 3650 50  0001 C CNN
+F 0 "#PWR07" H 7050 3650 50  0001 C CNN
 F 1 "+12V" H 7050 3940 50  0000 C CNN
 F 2 "" H 7050 3800 50  0001 C CNN
@@
 	7050 3800 7400 3800
 $Comp
-L GND #PWR014
+L GND #PWR08
 U 1 1 5B158127
 P 3700 2500
-F 0 "#PWR014" H 3700 2250 50  0001 C CNN
+F 0 "#PWR08" H 3700 2250 50  0001 C CNN
 F 1 "GND" H 3700 2350 50  0000 C CNN
 F 2 "" H 3700 2500 50  0001 C CNN
@@
 	2500 2000 2750 2000
 $Comp
-L Q_NMOS_GDS Q?
+L Q_NMOS_GDS Q2
 U 1 1 5B1583C2
 P 3600 3950
-F 0 "Q?" H 3800 4000 50  0000 L CNN
+F 0 "Q2" H 3800 4000 50  0000 L CNN
 F 1 "FQP30N06L" H 3800 3900 50  0000 L CNN
-F 2 "" H 3800 4050 50  0001 C CNN
+F 2 "TO_SOT_Packages_THT:TO-220-3_Vertical" H 3800 4050 50  0001 C CNN
 F 3 "" H 3600 3950 50  0001 C CNN
 	1    3600 3950
@@
 $EndComp
 $Comp
-L R R?
+L R R2
 U 1 1 5B1583C8
 P 2900 3950
-F 0 "R?" V 2980 3950 50  0000 C CNN
+F 0 "R2" V 2980 3950 50  0000 C CNN
 F 1 "100R" V 2900 3950 50  0000 C CNN
-F 2 "" V 2830 3950 50  0001 C CNN
+F 2 "Resistors_SMD:R_0805_HandSoldering" V 2830 3950 50  0001 C CNN
 F 3 "" H 2900 3950 50  0001 C CNN
 	1    2900 3950
@@
 $EndComp
 $Comp
-L R R?
+L R R5
 U 1 1 5B1583CE
 P 3200 4250
-F 0 "R?" V 3280 4250 50  0000 C CNN
+F 0 "R5" V 3280 4250 50  0000 C CNN
 F 1 "10K" V 3200 4250 50  0000 C CNN
-F 2 "" V 3130 4250 50  0001 C CNN
+F 2 "Resistors_SMD:R_0805_HandSoldering" V 3130 4250 50  0001 C CNN
 F 3 "" H 3200 4250 50  0001 C CNN
 	1    3200 4250
@@
 Connection ~ 3200 3950
 $Comp
-L GND #PWR015
+L GND #PWR09
 U 1 1 5B1583D7
 P 3700 4450
-F 0 "#PWR015" H 3700 4200 50  0001 C CNN
+F 0 "#PWR09" H 3700 4200 50  0001 C CNN
 F 1 "GND" H 3700 4300 50  0000 C CNN
 F 2 "" H 3700 4450 50  0001 C CNN
@@
 	2500 3950 2750 3950
 $Comp
-L Q_NMOS_GDS Q?
+L Q_NMOS_GDS Q3
 U 1 1 5B158B44
 P 3650 5750
-F 0 "Q?" H 3850 5800 50  0000 L CNN
+F 0 "Q3" H 3850 5800 50  0000 L CNN
 F 1 "FQP30N06L" H 3850 5700 50  0000 L CNN
-F 2 "" H 3850 5850 50  0001 C CNN
+F 2 "TO_SOT_Packages_THT:TO-220-3_Vertical" H 3850 5850 50  0001 C CNN
 F 3 "" H 3650 5750 50  0001 C CNN
 	1    3650 5750
@@
 $EndComp
 $Comp
-L R R?
+L R R3
 U 1 1 5B158B4A
 P 2950 5750
-F 0 "R?" V 3030 5750 50  0000 C CNN
+F 0 "R3" V 3030 5750 50  0000 C CNN
 F 1 "100R" V 2950 5750 50  0000 C CNN
-F 2 "" V 2880 5750 50  0001 C CNN
+F 2 "Resistors_SMD:R_0805_HandSoldering" V 2880 5750 50  0001 C CNN
 F 3 "" H 2950 5750 50  0001 C CNN
 	1    2950 5750
@@
 $EndComp
 $Comp
-L R R?
+L R R6
 U 1 1 5B158B50
 P 3250 6050
-F 0 "R?" V 3330 6050 50  0000 C CNN
+F 0 "R6" V 3330 6050 50  0000 C CNN
 F 1 "10K" V 3250 6050 50  0000 C CNN
-F 2 "" V 3180 6050 50  0001 C CNN
+F 2 "Resistors_SMD:R_0805_HandSoldering" V 3180 6050 50  0001 C CNN
 F 3 "" H 3250 6050 50  0001 C CNN
 	1    3250 6050
@@
 Connection ~ 3250 5750
 $Comp
-L GND #PWR016
+L GND #PWR010
 U 1 1 5B158B59
 P 3750 6250
-F 0 "#PWR016" H 3750 6000 50  0001 C CNN
+F 0 "#PWR010" H 3750 6000 50  0001 C CNN
 F 1 "GND" H 3750 6100 50  0000 C CNN
 F 2 "" H 3750 6250 50  0001 C CNN

Commit message: Did a stuff
Parts:
- added J1, J2, J3: TEST_1P, Measurement_Points:Measurement_Point_Square-SMD-Pad_Small, symbol conn1:TEST_1P
- J4: renamed from J2; symbol Conn_01x04 -> conn1:Conn_01x04
- Q1: symbol Q_NMOS_GDS -> device1:Q_NMOS_GDS
- Q2: renamed from Q3; symbol Q_NMOS_GDS -> device1:Q_NMOS_GDS
- Q3: renamed from Q2; symbol Q_NMOS_GDS -> device1:Q_NMOS_GDS
- R1, R4: symbol R -> device1:R
- R2: renamed from R3; symbol R -> device1:R
- R3: renamed from R2; symbol R -> device1:R
- R5: renamed from R6; symbol R -> device1:R
- R6: renamed from R5; symbol R -> device1:R
Connections:
- wire segments 22 -> 34

Commit message: changed some parts to smd, fixed some design errors
Parts:
- removed Q2, Q3: FQP30N06L, TO_SOT_Packages_THT:TO-220-3_Vertical, symbol device1:Q_NMOS_GDS
- added J8: Conn_01x04, Connector_PinHeader_2.54mm:PinHeader_1x04_P2.54mm_Vertical, symbol leddings-rescue:Conn_01x04-conn1
- added Q2, Q3: IRLR8726TRLPBF, Package_TO_SOT_SMD:TO-252-2, symbol leddings-rescue:Q_NMOS_GDS-device1
- J1, J2, J3: symbol conn1:TEST_1P -> leddings-rescue:TEST_1P-conn1
- J4: footprint Pin_Headers:Pin_Header_Straight_1x04_Pitch2.54mm -> TerminalBlock:TerminalBlock_bornier-4_P5.08mm; symbol conn1:Conn_01x04 -> leddings-rescue:Conn_01x04-conn1
- Q1: value FQP30N06L -> IRLR8726TRLPBF; footprint TO_SOT_Packages_THT:TO-220-3_Vertical -> Package_TO_SOT_SMD:TO-252-2; symbol device1:Q_NMOS_GDS -> leddings-rescue:Q_NMOS_GDS-device1
- R1, R2, R3, R4, R5, R6: symbol device1:R -> leddings-rescue:R-device1
Connections:
- wire segments 34 -> 54
Changed lines of the file:
@@
 $EndDescr
 $Comp
-L device1:Q_NMOS_GDS Q1
+L leddings-rescue:Q_NMOS_GDS-device1 Q1
 U 1 1 5B157B68
 P 3600 2000
 F 0 "Q1" H 3800 2050 50  0000 L CNN
-F 1 "FQP30N06L" H 3800 1950 50  0000 L CNN
-F 2 "TO_SOT_Packages_THT:TO-220-3_Vertical" H 3800 2100 50  0001 C CNN
+F 1 "IRLR8726TRLPBF" H 3800 1950 50  0000 L CNN
+F 2 "Package_TO_SOT_SMD:TO-252-2" H 3800 2100 50  0001 C CNN
 F 3 "" H 3600 2000 50  0001 C CNN
 	1    3600 2000
@@
 $EndComp
 $Comp
-L device1:R R1
+L leddings-rescue:R-device1 R1
 U 1 1 5B157EE6
 P 2900 2000
@@
 $EndComp
 $Comp
-L device1:R R4
+L leddings-rescue:R-device1 R4
 U 1 1 5B157F0E
 P 3200 2300
@@
 	3200 2150 3200 2000
 Connection ~ 3200 2000
-Text Label 7050 3500 2    60   ~ 0
+Text Label 7050 3600 2    60   ~ 0
 GreenChannel
-Text Label 7050 3600 2    60   ~ 0
+Text Label 7050 3700 2    60   ~ 0
 BlueChannel
-Text Label 7050 3700 2    60   ~ 0
+Text Label 7050 3800 2    60   ~ 0
 RedChannel
 Wire Wire Line
-	7050 3500 7400 3500
-Wire Wire Line
-	7400 3600 7050 3600
-Wire Wire Line
-	7050 3700 7400 3700
-$Comp
-L conn1:Conn_01x04 J4
+	7050 3700 7350 3700
+$Comp
+L leddings-rescue:Conn_01x04-conn1 J4
 U 1 1 5B158040
 P 7600 3600
 F 0 "J4" H 7600 3800 50  0000 C CNN
 F 1 "Conn_01x04" H 7600 3300 50  0000 C CNN
-F 2 "Pin_Headers:Pin_Header_Straight_1x04_Pitch2.54mm" H 7600 3600 50  0001 C CNN
+F 2 "TerminalBlock:TerminalBlock_bornier-4_P5.08mm" H 7600 3600 50  0001 C CNN
 F 3 "" H 7600 3600 50  0001 C CNN
 	1    7600 3600
@@
 L power1:+12V #PWR07
 U 1 1 5B1580E3
-P 7050 3800
-F 0 "#PWR07" H 7050 3650 50  0001 C CNN
-F 1 "+12V" H 7050 3940 50  0000 C CNN
-F 2 "" H 7050 3800 50  0001 C CNN
-F 3 "" H 7050 3800 50  0001 C CNN
-	1    7050 3800
+P 7050 3500
+F 0 "#PWR07" H 7050 3350 50  0001 C CNN
+F 1 "+12V" H 7050 3640 50  0000 C CNN
+F 2 "" H 7050 3500 50  0001 C CNN
+F 3 "" H 7050 3500 50  0001 C CNN
+	1    7050 3500
 	0    -1   -1   0
 $EndComp
 Wire Wire Line
-	7050 3800 7400 3800
+	7050 3800 7250 3800
 $Comp
 L power1:GND #PWR08
@@
 	2500 2000 2650 2000
 $Comp
-L device1:Q_NMOS_GDS Q3
-U 1 1 5B1583C2
-P 3650 5600
-F 0 "Q3" H 3850 5650 50  0000 L CNN
-F 1 "FQP30N06L" H 3850 5550 50  0000 L CNN
-F 2 "TO_SOT_Packages_THT:TO-220-3_Vertical" H 3850 5700 50  0001 C CNN
-F 3 "" H 3650 5600 50  0001 C CNN
-	1    3650 5600
-	1    0    0    -1
-$EndComp
-$Comp
-L device1:R R3
+L leddings-rescue:R-device1 R3
 U 1 1 5B1583C8
 P 2950 5600
@@
 $EndComp
 $Comp
-L device1:R R6
+L leddings-rescue:R-device1 R6
 U 1 1 5B1583CE
 P 3250 5900
@@
 	2550 5600 2650 5600
 $Comp
-L device1:Q_NMOS_GDS Q2
-U 1 1 5B158B44
-P 3600 3850
-F 0 "Q2" H 3800 3900 50  0000 L CNN
-F 1 "FQP30N06L" H 3800 3800 50  0000 L CNN
-F 2 "TO_SOT_Packages_THT:TO-220-3_Vertical" H 3800 3950 50  0001 C CNN
-F 3 "" H 3600 3850 50  0001 C CNN
-	1    3600 3850
-	1    0    0    -1
-$EndComp
-$Comp
-L device1:R R2
+L leddings-rescue:R-device1 R2
 U 1 1 5B158B4A
 P 2900 3850
@@
 $EndComp
 $Comp
-L device1:R R5
+L leddings-rescue:R-device1 R5
 U 1 1 5B158B50
 P 3200 4150
@@
 	3700 4300 3700 4350
 $Comp
-L conn1:TEST_1P J1
+L leddings-rescue:TEST_1P-conn1 J1
 U 1 1 5B4FC570
 P 2650 2150
@@
 $EndComp
 $Comp
-L conn1:TEST_1P J3
+L leddings-rescue:TEST_1P-conn1 J3
 U 1 1 5B4FC66D
 P 2650 5750
@@
 $EndComp
 $Comp
-L conn1:TEST_1P J2
+L leddings-rescue:TEST_1P-conn1 J2
 U 1 1 5B4FC771
 P 2600 4000
@@
 Wire Wire Line
 	2600 3850 2750 3850
+$Comp
+L leddings-rescue:Conn_01x04-conn1 J8
+U 1 1 5BF8470A
+P 8200 3600
+F 0 "J8" H 8200 3800 50  0000 C CNN
+F 1 "Conn_01x04" H 8200 3300 50  0000 C CNN
+F 2 "Connector_PinHeader_2.54mm:PinHeader_1x04_P2.54mm_Vertical" H 8200 3600 50  0001 C CNN
+F 3 "" H 8200 3600 50  0001 C CNN
+	1    8200 3600
+	1    0    0    -1
+$EndComp
+Wire Wire Line
+	7850 3500 8000 3500
+Wire Wire Line
+	7350 3700 7350 4000
+Wire Wire Line
+	7350 4000 7750 4000
+Wire Wire Line
+	7750 4000 7750 3700
+Wire Wire Line
+	7750 3700 8000 3700
+Connection ~ 7350 3700
+Wire Wire Line
+	7350 3700 7400 3700
+Wire Wire Line
+	8000 3800 7850 3800
+Wire Wire Line
+	7850 3800 7850 4100
+Wire Wire Line
+	7850 4100 7250 4100
+Wire Wire Line
+	7250 4100 7250 3800
+Connection ~ 7250 3800
+Wire Wire Line
+	7250 3800 7400 3800
+Wire Wire Line
+	7050 3600 7350 3600
+Wire Wire Line
+	7050 3500 7250 3500
+Wire Wire Line
+	7750 3600 7750 3350
+Wire Wire Line
+	7750 3350 7350 3350
+Wire Wire Line
+	7350 3350 7350 3600
+Wire Wire Line
+	7750 3600 8000 3600
+Connection ~ 7350 3600
+Wire Wire Line
+	7350 3600 7400 3600
+Wire Wire Line
+	7850 3250 7250 3250
+Wire Wire Line
+	7250 3250 7250 3500
+Wire Wire Line
+	7850 3250 7850 3500
+Connection ~ 7250 3500
+Wire Wire Line
+	7250 3500 7400 3500
+$Comp
+L leddings-rescue:Q_NMOS_GDS-device1 Q2
+U 1 1 5BF8968B
+P 3600 3850
+F 0 "Q2" H 3800 3900 50  0000 L CNN
+F 1 "IRLR8726TRLPBF" H 3800 3800 50  0000 L CNN
+F 2 "Package_TO_SOT_SMD:TO-252-2" H 3800 3950 50  0001 C CNN
+F 3 "" H 3600 3850 50  0001 C CNN
+	1    3600 3850
+	1    0    0    -1
+$EndComp
+$Comp
+L leddings-rescue:Q_NMOS_GDS-device1 Q3
+U 1 1 5BF899AF
+P 3650 5600
+F 0 "Q3" H 3850 5650 50  0000 L CNN
+F 1 "IRLR8726TRLPBF" H 3850 5550 50  0000 L CNN
+F 2 "Package_TO_SOT_SMD:TO-252-2" H 3850 5700 50  0001 C CNN
+F 3 "" H 3650 5600 50  0001 C CNN
+	1    3650 5600
+	1    0    0    -1
+$EndComp
 $EndSCHEMATC
