File: power.sch (KiCad schematic (older format))
At the start: 5 parts

Commit message: added stuff
Parts:
- C1, C2: renamed from C?; footprint (none) -> Capacitors_SMD:C_0805_HandSoldering
- D1: renamed from D?; footprint (none) -> Diodes_SMD:D_0805
- gave numbers to parts that had none: 2
Changed lines of the file:
@@
 $EndDescr
 $Comp
-L VBUS #PWR07
+L VBUS #PWR01
 U 1 1 5B1573D9
 P 6200 3200
-F 0 "#PWR07" H 6200 3050 50  0001 C CNN
+F 0 "#PWR01" H 6200 3050 50  0001 C CNN
 F 1 "VBUS" H 6200 3350 50  0000 C CNN
 F 2 "" H 6200 3200 50  0001 C CNN
@@
 $EndComp
 $Comp
-L +12V #PWR08
+L +12V #PWR02
 U 1 1 5B1573DF
 P 5850 3450
-F 0 "#PWR08" H 5850 3300 50  0001 C CNN
+F 0 "#PWR02" H 5850 3300 50  0001 C CNN
 F 1 "+12V" H 5850 3590 50  0000 C CNN
 F 2 "" H 5850 3450 50  0001 C CNN
@@
 $EndComp
 $Comp
-L GND #PWR09
+L GND #PWR03
 U 1 1 5B1573E5
 P 6950 4700
-F 0 "#PWR09" H 6950 4450 50  0001 C CNN
+F 0 "#PWR03" H 6950 4450 50  0001 C CNN
 F 1 "GND" H 6950 4550 50  0000 C CNN
 F 2 "" H 6950 4700 50  0001 C CNN
@@
 $EndComp
 $Comp
-L D D?
+L D D1
 U 1 1 5B1573F2
 P 6200 3450
-F 0 "D?" H 6200 3550 50  0000 C CNN
+F 0 "D1" H 6200 3550 50  0000 C CNN
 F 1 "D" H 6200 3350 50  0000 C CNN
-F 2 "" H 6200 3450 50  0001 C CNN
+F 2 "Diodes_SMD:D_0805" H 6200 3450 50  0001 C CNN
 F 3 "" H 6200 3450 50  0001 C CNN
 	1    6200 3450
@@
 	6950 4000 6950 4700
 $Comp
-L VCC #PWR010
+L VCC #PWR04
 U 1 1 5B157413
 P 8250 3700
-F 0 "#PWR010" H 8250 3550 50  0001 C CNN
+F 0 "#PWR04" H 8250 3550 50  0001 C CNN
 F 1 "VCC" H 8250 3850 50  0000 C CNN
 F 2 "" H 8250 3700 50  0001 C CNN
@@
 	7850 4550 7850 4100
 $Comp
-L Barrel_Jack J?
+L Barrel_Jack J1
 U 1 1 5B1577C1
 P 2550 3450
-F 0 "J?" H 2550 3660 50  0000 C CNN
+F 0 "J1" H 2550 3660 50  0000 C CNN
 F 1 "Barrel_Jack" H 2550 3275 50  0000 C CNN
 F 2 "" H 2600 3410 50  0001 C CNN
@@
 $EndComp
 $Comp
-L +12V #PWR011
+L +12V #PWR05
 U 1 1 5B15783A
 P 3150 3350
-F 0 "#PWR011" H 3150 3200 50  0001 C CNN
+F 0 "#PWR05" H 3150 3200 50  0001 C CNN
 F 1 "+12V" H 3150 3490 50  0000 C CNN
 F 2 "" H 3150 3350 50  0001 C CNN
@@
 $EndComp
 $Comp
-L GND #PWR012
+L GND #PWR06
 U 1 1 5B15785A
 P 3150 3550
-F 0 "#PWR012" H 3150 3300 50  0001 C CNN
+F 0 "#PWR06" H 3150 3300 50  0001 C CNN
 F 1 "GND" H 3150 3400 50  0000 C CNN
 F 2 "" H 3150 3550 50  0001 C CNN
@@
 	2850 3350 3150 3350
 $Comp
-L LM1117-3.3 U?
+L LM1117-3.3 U1
 U 1 1 5B194466
 P 6950 3700
-F 0 "U?" H 6800 3825 50  0000 C CNN
+F 0 "U1" H 6800 3825 50  0000 C CNN
 F 1 "LM1117-3.3" H 6950 3825 50  0000 L CNN
 F 2 "TO_SOT_Packages_THT:TO-220-3_Vertical" H 6950 3700 50  0001 C CNN
@@
 $EndComp
 $Comp
-L C C?
+L C C2
 U 1 1 5B157419
 P 7850 3950
-F 0 "C?" H 7875 4050 50  0000 L CNN
+F 0 "C2" H 7875 4050 50  0000 L CNN
 F 1 "10uF" H 7875 3850 50  0000 L CNN
-F 2 "" H 7888 3800 50  0001 C CNN
+F 2 "Capacitors_SMD:C_0805_HandSoldering" H 7888 3800 50  0001 C CNN
 F 3 "" H 7850 3950 50  0001 C CNN
 	1    7850 3950
@@
 $EndComp
 $Comp
-L C C?
+L C C1
 U 1 1 5B19450F
 P 6200 3950
-F 0 "C?" H 6225 4050 50  0000 L CNN
+F 0 "C1" H 6225 4050 50  0000 L CNN
 F 1 "10uF" H 6225 3850 50  0000 L CNN
-F 2 "" H 6238 3800 50  0001 C CNN
+F 2 "Capacitors_SMD:C_0805_HandSoldering" H 6238 3800 50  0001 C CNN
 F 3 "" H 6200 3950 50  0001 C CNN
 	1    6200 3950

Commit message: Did a stuff
Parts:
- added MK1, MK2, MK3, MK4: Mounting_Hole, Mounting_Holes:MountingHole_3.2mm_M3_DIN965_Pad, symbol mechanical1:Mounting_Hole
- C1, C2: symbol C -> device1:C
- D1: symbol D -> device1:D
- J6: renamed from J1; footprint (none) -> Connectors:Barrel_Jack_CUI_PJ-102AH; symbol Barrel_Jack -> conn1:Barrel_Jack
- U1: symbol LM1117-3.3 -> regul1:LM1117-3.3
Connections:
- wire segments 14 -> 20
Changed lines of the file:
@@
-EESchema Schematic File Version 2
-LIBS:power
-LIBS:device
-LIBS:switches
-LIBS:relays
-LIBS:motors
-LIBS:transistors
-LIBS:conn
-LIBS:linear
-LIBS:regul
-LIBS:74xx
-LIBS:cmos4000
-LIBS:adc-dac
-LIBS:memory
-LIBS:xilinx
-LIBS:microcontrollers
-LIBS:dsp
-LIBS:microchip
-LIBS:analog_switches
-LIBS:motorola
-LIBS:texas
-LIBS:intel
-LIBS:audio
-LIBS:interface
-LIBS:digital-audio
-LIBS:philips
-LIBS:display
-LIBS:cypress
-LIBS:siliconi
-LIBS:opto
-LIBS:atmel
-LIBS:contrib
-LIBS:valves
-LIBS:ESP8266
-LIBS:74xgxx
-LIBS:ac-dc
-LIBS:actel
-LIBS:allegro
-LIBS:Altera
-LIBS:analog_devices
-LIBS:battery_management
-LIBS:bbd
-LIBS:bosch
-LIBS:brooktre
-LIBS:cmos_ieee
-LIBS:dc-dc
-LIBS:diode
-LIBS:elec-unifil
-LIBS:ESD_Protection
-LIBS:ftdi
-LIBS:gennum
-LIBS:graphic_symbols
-LIBS:hc11
-LIBS:infineon
-LIBS:intersil
-LIBS:ir
-LIBS:Lattice
-LIBS:leds
-LIBS:LEM
-LIBS:logic_programmable
-LIBS:maxim
-LIBS:mechanical
-LIBS:microchip_dspic33dsc
-LIBS:microchip_pic10mcu
-LIBS:microchip_pic12mcu
-LIBS:microchip_pic16mcu
-LIBS:microchip_pic18mcu
-LIBS:microchip_pic24mcu
-LIBS:microchip_pic32mcu
-LIBS:modules
-LIBS:motor_drivers
-LIBS:msp430
-LIBS:nordicsemi
-LIBS:nxp
-LIBS:nxp_armmcu
-LIBS:onsemi
-LIBS:Oscillators
-LIBS:powerint
-LIBS:Power_Management
-LIBS:pspice
-LIBS:references
-LIBS:rfcom
-LIBS:RFSolutions
-LIBS:sensors
-LIBS:silabs
-LIBS:stm8
-LIBS:stm32
-LIBS:supertex
-LIBS:transf
-LIBS:triac_thyristor
-LIBS:ttl_ieee
-LIBS:video
-LIBS:wiznet
-LIBS:Worldsemi
-LIBS:Xicor
-LIBS:zetex
-LIBS:Zilog
-LIBS:ch34x
+EESchema Schematic File Version 4
 LIBS:leddings-cache
-EELAYER 25 0
+EELAYER 26 0
 EELAYER END
 $Descr A4 11693 8268
@@
 $EndDescr
 $Comp
-L VBUS #PWR01
+L power1:VBUS #PWR01
 U 1 1 5B1573D9
 P 6200 3200
@@
 $EndComp
 $Comp
-L +12V #PWR02
+L power1:+12V #PWR02
 U 1 1 5B1573DF
 P 5850 3450
@@
 $EndComp
 $Comp
-L GND #PWR03
+L power1:GND #PWR03
 U 1 1 5B1573E5
 P 6950 4700
@@
 $EndComp
 $Comp
-L D D1
+L device1:D D1
 U 1 1 5B1573F2
 P 6200 3450
@@
 	5850 3450 5850 3700
 Wire Wire Line
-	5850 3700 6650 3700
-Wire Wire Line
-	6200 3600 6200 3800
+	5850 3700 6200 3700
+Wire Wire Line
+	6200 3600 6200 3700
 Connection ~ 6200 3700
 Wire Wire Line
-	7250 3700 8250 3700
-Wire Wire Line
-	6200 4550 7850 4550
-Wire Wire Line
-	6950 4000 6950 4700
-$Comp
-L VCC #PWR04
+	7250 3700 7850 3700
+Wire Wire Line
+	6200 4550 6950 4550
+Wire Wire Line
+	6950 4000 6950 4550
+$Comp
+L power1:VCC #PWR04
 U 1 1 5B157413
 P 8250 3700
@@
 	7850 4550 7850 4100
 $Comp
-L Barrel_Jack J1
+L conn1:Barrel_Jack J6
 U 1 1 5B1577C1
 P 2550 3450
-F 0 "J1" H 2550 3660 50  0000 C CNN
+F 0 "J6" H 2550 3660 50  0000 C CNN
 F 1 "Barrel_Jack" H 2550 3275 50  0000 C CNN
-F 2 "" H 2600 3410 50  0001 C CNN
+F 2 "Connectors:Barrel_Jack_CUI_PJ-102AH" H 2600 3410 50  0001 C CNN
 F 3 "" H 2600 3410 50  0001 C CNN
 	1    2550 3450
@@
 $EndComp
 $Comp
-L +12V #PWR05
+L power1:+12V #PWR05
 U 1 1 5B15783A
 P 3150 3350
@@
 $EndComp
 $Comp
-L GND #PWR06
+L power1:GND #PWR06
 U 1 1 5B15785A
 P 3150 3550
@@
 	3000 3450 3000 3550
 Wire Wire Line
-	2850 3550 3150 3550
+	2850 3550 3000 3550
 Connection ~ 3000 3550
 Wire Wire Line
 	2850 3350 3150 3350
 $Comp
-L LM1117-3.3 U1
+L regul1:LM1117-3.3 U1
 U 1 1 5B194466
 P 6950 3700
@@
 $EndComp
 $Comp
-L C C2
+L device1:C C2
 U 1 1 5B157419
 P 7850 3950
@@
 $EndComp
 $Comp
-L C C1
+L device1:C C1
 U 1 1 5B19450F
 P 6200 3950
@@
 	6200 4100 6200 4550
 Connection ~ 6950 4550
+Wire Wire Line
+	6200 3700 6650 3700
+Wire Wire Line
+	6200 3700 6200 3800
+Wire Wire Line
+	7850 3700 8250 3700
+Wire Wire Line
+	3000 3550 3150 3550
+Wire Wire Line
+	6950 4550 7850 4550
+Wire Wire Line
+	6950 4550 6950 4700
+$Comp
+L mechanical1:Mounting_Hole MK4
+U 1 1 5B4FC85C
+P 8850 1650
+F 0 "MK4" H 8950 1696 50  0000 L CNN
+F 1 "Mounting_Hole" H 8950 1605 50  0000 L CNN
+F 2 "Mounting_Holes:MountingHole_3.2mm_M3_DIN965_Pad" H 8850 1650 50  0001 C CNN
+F 3 "" H 8850 1650 50  0001 C CNN
+	1    8850 1650
+	1    0    0    -1
+$EndComp
+$Comp
+L mechanical1:Mounting_Hole MK3
+U 1 1 5B4FCD04
+P 8700 1100
+F 0 "MK3" H 8800 1146 50  0000 L CNN
+F 1 "Mounting_Hole" H 8800 1055 50  0000 L CNN
+F 2 "Mounting_Holes:MountingHole_3.2mm_M3_DIN965_Pad" H 8700 1100 50  0001 C CNN
+F 3 "" H 8700 1100 50  0001 C CNN
+	1    8700 1100
+	1    0    0    -1
+$EndComp
+$Comp
+L mechanical1:Mounting_Hole MK2
+U 1 1 5B4FCECE
+P 7950 1600
+F 0 "MK2" H 8050 1646 50  0000 L CNN
+F 1 "Mounting_Hole" H 8050 1555 50  0000 L CNN
+F 2 "Mounting_Holes:MountingHole_3.2mm_M3_DIN965_Pad" H 7950 1600 50  0001 C CNN
+F 3 "" H 7950 1600 50  0001 C CNN
+	1    7950 1600
+	1    0    0    -1
+$EndComp
+$Comp
+L mechanical1:Mounting_Hole MK1
+U 1 1 5B4FCED4
+P 7800 1050
+F 0 "MK1" H 7900 1096 50  0000 L CNN
+F 1 "Mounting_Hole" H 7900 1005 50  0000 L CNN
+F 2 "Mounting_Holes:MountingHole_3.2mm_M3_DIN965_Pad" H 7800 1050 50  0001 C CNN
+F 3 "" H 7800 1050 50  0001 C CNN
+	1    7800 1050
+	1    0    0    -1
+$EndComp
 $EndSCHEMATC

Commit message: added pin headers for uart, added power-on-led, improved routing
Parts:
- added D2: LED, LEDs:LED_0805_HandSoldering, symbol Device:LED
- added R9: 1K, Resistors_SMD:R_0805_HandSoldering, symbol Device:R
Connections:
- wire segments 20 -> 25
Changed lines of the file:
@@
 encoding utf-8
 Sheet 2 5
-Title ""
-Date ""
-Rev ""
+Title "LED Driver"
+Date "2018-10-02"
+Rev "1.0"
 Comp ""
 Comment1 ""
@@
 L power1:VCC #PWR04
 U 1 1 5B157413
-P 8250 3700
-F 0 "#PWR04" H 8250 3550 50  0001 C CNN
-F 1 "VCC" H 8250 3850 50  0000 C CNN
-F 2 "" H 8250 3700 50  0001 C CNN
-F 3 "" H 8250 3700 50  0001 C CNN
-	1    8250 3700
+P 9500 3700
+F 0 "#PWR04" H 9500 3550 50  0001 C CNN
+F 1 "VCC" H 9500 3850 50  0000 C CNN
+F 2 "" H 9500 3700 50  0001 C CNN
+F 3 "" H 9500 3700 50  0001 C CNN
+	1    9500 3700
 	0    1    1    0
 $EndComp
@@
 	6200 3700 6200 3800
 Wire Wire Line
-	7850 3700 8250 3700
+	7850 3700 8850 3700
 Wire Wire Line
 	3000 3550 3150 3550
@@
 	1    0    0    -1
 $EndComp
+$Comp
+L Device:LED D2
+U 1 1 5BB3B41C
+P 8850 4350
+F 0 "D2" V 8888 4233 50  0000 R CNN
+F 1 "LED" V 8797 4233 50  0000 R CNN
+F 2 "LEDs:LED_0805_HandSoldering" H 8850 4350 50  0001 C CNN
+F 3 "~" H 8850 4350 50  0001 C CNN
+	1    8850 4350
+	0    -1   -1   0
+$EndComp
+$Comp
+L Device:R R9
+U 1 1 5BB3B508
+P 8850 3950
+F 0 "R9" H 8920 3996 50  0000 L CNN
+F 1 "1K" H 8920 3905 50  0000 L CNN
+F 2 "Resistors_SMD:R_0805_HandSoldering" V 8780 3950 50  0001 C CNN
+F 3 "~" H 8850 3950 50  0001 C CNN
+	1    8850 3950
+	1    0    0    -1
+$EndComp
+Wire Wire Line
+	8850 3800 8850 3700
+Connection ~ 8850 3700
+Wire Wire Line
+	8850 3700 9500 3700
+Wire Wire Line
+	8850 4200 8850 4100
+Wire Wire Line
+	7850 4550 8850 4550
+Wire Wire Line
+	8850 4550 8850 4500
+Connection ~ 7850 4550
 $EndSCHEMATC

Commit message: changed some parts to smd, fixed some design errors
Parts:
- C1, C2: symbol device1:C -> leddings-rescue:C-device1
- D1: footprint Diodes_SMD:D_0805 -> Diode_SMD:D_SOD-123F; symbol device1:D -> leddings-rescue:D-device1
- J6: symbol conn1:Barrel_Jack -> leddings-rescue:Barrel_Jack-conn1
- MK1, MK2, MK3, MK4: symbol mechanical1:Mounting_Hole -> leddings-rescue:Mounting_Hole-mechanical1
- R9: value 1K -> 10K
- U1: footprint TO_SOT_Packages_THT:TO-220-3_Vertical -> Package_TO_SOT_SMD:TO-252-2; symbol regul1:LM1117-3.3 -> leddings-rescue:LM1117-3.3-regul1
Changed lines of the file:
@@
 $EndComp
 $Comp
-L device1:D D1
+L leddings-rescue:D-device1 D1
 U 1 1 5B1573F2
 P 6200 3450
 F 0 "D1" H 6200 3550 50  0000 C CNN
 F 1 "D" H 6200 3350 50  0000 C CNN
-F 2 "Diodes_SMD:D_0805" H 6200 3450 50  0001 C CNN
+F 2 "Diode_SMD:D_SOD-123F" H 6200 3450 50  0001 C CNN
 F 3 "" H 6200 3450 50  0001 C CNN
 	1    6200 3450
@@
 	7850 4550 7850 4100
 $Comp
-L conn1:Barrel_Jack J6
+L leddings-rescue:Barrel_Jack-conn1 J6
 U 1 1 5B1577C1
 P 2550 3450
+AR Path="/5B1577C1" Ref="J6"  Part="1"
+AR Path="/5B156FC6/5B1577C1" Ref="J6"  Part="1"
 F 0 "J6" H 2550 3660 50  0000 C CNN
 F 1 "Barrel_Jack" H 2550 3275 50  0000 C CNN
@@
 	2850 3350 3150 3350
 $Comp
-L regul1:LM1117-3.3 U1
+L leddings-rescue:LM1117-3.3-regul1 U1
 U 1 1 5B194466
 P 6950 3700
 F 0 "U1" H 6800 3825 50  0000 C CNN
 F 1 "LM1117-3.3" H 6950 3825 50  0000 L CNN
-F 2 "TO_SOT_Packages_THT:TO-220-3_Vertical" H 6950 3700 50  0001 C CNN
+F 2 "Package_TO_SOT_SMD:TO-252-2" H 6950 3700 50  0001 C CNN
 F 3 "" H 6950 3700 50  0001 C CNN
 	1    6950 3700
@@
 $EndComp
 $Comp
-L device1:C C2
+L leddings-rescue:C-device1 C2
 U 1 1 5B157419
 P 7850 3950
@@
 $EndComp
 $Comp
-L device1:C C1
+L leddings-rescue:C-device1 C1
 U 1 1 5B19450F
 P 6200 3950
@@
 	6950 4550 6950 4700
 $Comp
-L mechanical1:Mounting_Hole MK4
+L leddings-rescue:Mounting_Hole-mechanical1 MK4
 U 1 1 5B4FC85C
 P 8850 1650
@@
 $EndComp
 $Comp
-L mechanical1:Mounting_Hole MK3
+L leddings-rescue:Mounting_Hole-mechanical1 MK3
 U 1 1 5B4FCD04
 P 8700 1100
@@
 $EndComp
 $Comp
-L mechanical1:Mounting_Hole MK2
+L leddings-rescue:Mounting_Hole-mechanical1 MK2
 U 1 1 5B4FCECE
 P 7950 1600
@@
 $EndComp
 $Comp
-L mechanical1:Mounting_Hole MK1
+L leddings-rescue:Mounting_Hole-mechanical1 MK1
 U 1 1 5B4FCED4
 P 7800 1050
@@
 P 8850 3950
 F 0 "R9" H 8920 3996 50  0000 L CNN
-F 1 "1K" H 8920 3905 50  0000 L CNN
+F 1 "10K" H 8920 3905 50  0000 L CNN
 F 2 "Resistors_SMD:R_0805_HandSoldering" V 8780 3950 50  0001 C CNN
 F 3 "~" H 8850 3950 50  0001 C CNN
