File: smarts.sch (KiCad schematic (older format))
At the start: 5 parts, among them SW1 SW_RESET, SW2 Boot SEL, U3 ESP-07v2

Commit message: Did a stuff
Parts:
- removed U3: ESP-07v2, RF_Modules:ESP-12E, symbol ESP-07v2
- added U3: ESP-12E, ESP8266:ESP-12E_SMD, symbol ESP8266:ESP-12E
- R7, R8: symbol R -> device1:R
- SW1: symbol SW_Push -> switches1:SW_Push
- SW2: footprint Connectors:GS3 -> Pin_Headers:Pin_Header_Straight_1x03_Pitch1.27mm; symbol GS3 -> conn1:GS3
Connections:
- wire segments 21 -> 30
- no-connect marks 6 -> 12
Changed lines of the file:
@@
-EESchema Schematic File Version 2
-LIBS:power
-LIBS:device
-LIBS:switches
-LIBS:relays
-LIBS:motors
-LIBS:transistors
-LIBS:conn
-LIBS:linear
-LIBS:regul
-LIBS:74xx
-LIBS:cmos4000
-LIBS:adc-dac
-LIBS:memory
-LIBS:xilinx
-LIBS:microcontrollers
-LIBS:dsp
-LIBS:microchip
-LIBS:analog_switches
-LIBS:motorola
-LIBS:texas
-LIBS:intel
-LIBS:audio
-LIBS:interface
-LIBS:digital-audio
-LIBS:philips
-LIBS:display
-LIBS:cypress
-LIBS:siliconi
-LIBS:opto
-LIBS:atmel
-LIBS:contrib
-LIBS:valves
-LIBS:ESP8266
-LIBS:74xgxx
-LIBS:ac-dc
-LIBS:actel
-LIBS:allegro
-LIBS:Altera
-LIBS:analog_devices
-LIBS:battery_management
-LIBS:bbd
-LIBS:bosch
-LIBS:brooktre
-LIBS:cmos_ieee
-LIBS:dc-dc
-LIBS:diode
-LIBS:elec-unifil
-LIBS:ESD_Protection
-LIBS:ftdi
-LIBS:gennum
-LIBS:graphic_symbols
-LIBS:hc11
-LIBS:infineon
-LIBS:intersil
-LIBS:ir
-LIBS:Lattice
-LIBS:leds
-LIBS:LEM
-LIBS:logic_programmable
-LIBS:maxim
-LIBS:mechanical
-LIBS:microchip_dspic33dsc
-LIBS:microchip_pic10mcu
-LIBS:microchip_pic12mcu
-LIBS:microchip_pic16mcu
-LIBS:microchip_pic18mcu
-LIBS:microchip_pic24mcu
-LIBS:microchip_pic32mcu
-LIBS:modules
-LIBS:motor_drivers
-LIBS:msp430
-LIBS:nordicsemi
-LIBS:nxp
-LIBS:nxp_armmcu
-LIBS:onsemi
-LIBS:Oscillators
-LIBS:powerint
-LIBS:Power_Management
-LIBS:pspice
-LIBS:references
-LIBS:rfcom
-LIBS:RFSolutions
-LIBS:sensors
-LIBS:silabs
-LIBS:stm8
-LIBS:stm32
-LIBS:supertex
-LIBS:transf
-LIBS:triac_thyristor
-LIBS:ttl_ieee
-LIBS:video
-LIBS:wiznet
-LIBS:Worldsemi
-LIBS:Xicor
-LIBS:zetex
-LIBS:Zilog
-LIBS:ch34x
+EESchema Schematic File Version 4
 LIBS:leddings-cache
-EELAYER 25 0
+EELAYER 26 0
 EELAYER END
 $Descr A4 11693 8268
@@
 $EndDescr
 $Comp
-L ESP-07v2 U3
-U 1 1 5B193085
-P 5150 4150
-F 0 "U3" H 5150 4050 50  0000 C CNN
-F 1 "ESP-07v2" H 5150 4250 50  0000 C CNN
-F 2 "RF_Modules:ESP-12E" H 5150 4150 50  0001 C CNN
-F 3 "" H 5150 4150 50  0001 C CNN
-	1    5150 4150
-	1    0    0    -1
-$EndComp
-$Comp
-L SW_Push SW1
+L switches1:SW_Push SW1
 U 1 1 5B19308C
 P 3700 3850
@@
 $EndComp
 $Comp
-L R R7
+L device1:R R7
 U 1 1 5B193093
 P 4050 3550
@@
 	4050 3150 5150 3150
 Wire Wire Line
-	5150 2950 5150 3250
-Wire Wire Line
-	3900 3850 4250 3850
+	5150 2950 5150 3150
+Wire Wire Line
+	3900 3850 3950 3850
 Wire Wire Line
 	4050 3850 4050 3700
 Connection ~ 4050 3850
-Connection ~ 5150 3150
-$Comp
-L GND #PWR018
+$Comp
+L power1:GND #PWR018
 U 1 1 5B1930A1
 P 3300 3850
@@
 $EndComp
 Wire Wire Line
-	3300 3850 3500 3850
-$Comp
-L VCC #PWR019
+	3300 3850 3400 3850
+$Comp
+L power1:VCC #PWR019
 U 1 1 5B1930A8
 P 5150 2950
@@
 	1    0    0    -1
 $EndComp
-$Comp
-L GND #PWR020
-U 1 1 5B1930AE
-P 5150 5200
-F 0 "#PWR020" H 5150 4950 50  0001 C CNN
-F 1 "GND" H 5150 5050 50  0000 C CNN
-F 2 "" H 5150 5200 50  0001 C CNN
-F 3 "" H 5150 5200 50  0001 C CNN
-	1    5150 5200
-	1    0    0    -1
-$EndComp
-Wire Wire Line
-	5150 5200 5150 5050
 Wire Wire Line
 	4250 4050 3400 4050
@@
 Connection ~ 3400 3850
 $Comp
-L GS3 SW2
+L conn1:GS3 SW2
 U 1 1 5B1930B8
 P 7500 4250
 F 0 "SW2" H 7550 4450 50  0000 C CNN
 F 1 "Boot SEL" H 7550 4051 50  0000 C CNN
-F 2 "Connectors:GS3" V 7588 4176 50  0001 C CNN
+F 2 "Pin_Headers:Pin_Header_Straight_1x03_Pitch1.27mm" V 7588 4176 50  0001 C CNN
 F 3 "" H 7500 4250 50  0001 C CNN
 	1    7500 4250
@@
 $EndComp
 Wire Wire Line
-	6050 4250 7350 4250
-$Comp
-L GND #PWR021
+	6050 4250 6750 4250
+$Comp
+L power1:GND #PWR021
 U 1 1 5B1930C0
 P 7800 4350
@@
 $EndComp
 $Comp
-L VCC #PWR022
+L power1:VCC #PWR022
 U 1 1 5B1930C6
 P 7800 4150
@@
 	7800 4350 7650 4350
 $Comp
-L VCC #PWR023
+L power1:VCC #PWR023
 U 1 1 5B1930CE
 P 6750 3600
@@
 $EndComp
 $Comp
-L R R8
+L device1:R R8
 U 1 1 5B1930D4
 P 6750 3900
@@
 Connection ~ 6750 4250
 Wire Wire Line
-	3950 2400 3950 3850
+	3950 3450 3950 3850
 Connection ~ 3950 3850
 NoConn ~ 4250 3950
@@
 Text HLabel 6900 2850 1    60   Input ~ 0
 BOOT_SELECT
-Text HLabel 3950 2400 1    60   Input ~ 0
+Text HLabel 3500 3450 0    60   Input ~ 0
 RESET
 Text HLabel 6150 3850 2    60   Input ~ 0
@@
 Wire Wire Line
 	4150 4450 4250 4450
+Wire Wire Line
+	4050 3850 4250 3850
+Wire Wire Line
+	3400 3850 3500 3850
+Wire Wire Line
+	6750 4250 6900 4250
+Wire Wire Line
+	3950 3850 4050 3850
+Wire Wire Line
+	6900 4250 7350 4250
+$Comp
+L ESP8266:ESP-12E U3
+U 1 1 5B507C56
+P 5150 4150
+F 0 "U3" H 5150 4915 50  0000 C CNN
+F 1 "ESP-12E" H 5150 4824 50  0000 C CNN
+F 2 "ESP8266:ESP-12E_SMD" H 5150 4150 50  0001 C CNN
+F 3 "http://l0l.org.uk/2014/12/esp8266-modules-hardware-guide-gotta-catch-em-all/" H 5150 4150 50  0001 C CNN
+	1    5150 4150
+	1    0    0    -1
+$EndComp
+Wire Wire Line
+	4250 4550 2700 4550
+Wire Wire Line
+	2700 4550 2700 3150
+Wire Wire Line
+	2700 3150 4050 3150
+Connection ~ 4050 3150
+Wire Wire Line
+	3950 3450 3500 3450
+NoConn ~ 5400 5050
+NoConn ~ 5300 5050
+NoConn ~ 5200 5050
+NoConn ~ 5100 5050
+NoConn ~ 5000 5050
+NoConn ~ 4900 5050
+$Comp
+L power1:GND #PWR?
+U 1 1 5B50A811
+P 6200 4550
+F 0 "#PWR?" H 6200 4300 50  0001 C CNN
+F 1 "GND" V 6205 4422 50  0000 R CNN
+F 2 "" H 6200 4550 50  0001 C CNN
+F 3 "" H 6200 4550 50  0001 C CNN
+	1    6200 4550
+	0    -1   -1   0
+$EndComp
+Wire Wire Line
+	6050 4550 6200 4550
 $EndSCHEMATC

Commit message: ??
Changed lines of the file:
@@
 Text HLabel 4150 4250 0    60   Input ~ 0
 RED
+Text HLabel 4150 4450 0    60   Input ~ 0
+GREEN
 Text HLabel 4150 4350 0    60   Input ~ 0
-GREEN
-Text HLabel 4150 4450 0    60   Input ~ 0
 BLUE
 NoConn ~ 4250 4150
@@
 NoConn ~ 4900 5050
 $Comp
-L power1:GND #PWR?
+L power1:GND #PWR0101
 U 1 1 5B50A811
 P 6200 4550
-F 0 "#PWR?" H 6200 4300 50  0001 C CNN
+F 0 "#PWR0101" H 6200 4300 50  0001 C CNN
 F 1 "GND" V 6205 4422 50  0000 R CNN
 F 2 "" H 6200 4550 50  0001 C CNN

Commit message: added pin headers for uart, added power-on-led, improved routing
Parts:
- SW2: footprint Pin_Headers:Pin_Header_Straight_1x03_Pitch1.27mm -> Pin_Headers:Pin_Header_Straight_1x03_Pitch2.54mm
Changed lines of the file:
@@
 encoding utf-8
 Sheet 5 5
-Title ""
-Date ""
-Rev ""
+Title "LED Driver"
+Date "2018-10-02"
+Rev "1.0"
 Comp ""
 Comment1 ""
@@
 F 0 "SW2" H 7550 4450 50  0000 C CNN
 F 1 "Boot SEL" H 7550 4051 50  0000 C CNN
-F 2 "Pin_Headers:Pin_Header_Straight_1x03_Pitch1.27mm" V 7588 4176 50  0001 C CNN
+F 2 "Pin_Headers:Pin_Header_Straight_1x03_Pitch2.54mm" V 7588 4176 50  0001 C CNN
 F 3 "" H 7500 4250 50  0001 C CNN
 	1    7500 4250

Commit message: changed some parts to smd, fixed some design errors
Parts:
- added C6: 10uF, symbol Device:C
- R7, R8: symbol device1:R -> leddings-rescue:R-device1
- SW1: footprint Buttons_Switches_THT:SW_Tactile_Straight_KSA0Axx1LFTR -> Button_Switch_SMD:SW_SPST_B3S-1000; symbol switches1:SW_Push -> leddings-rescue:SW_Push-switches1
- SW2: symbol conn1:GS3 -> leddings-rescue:GS3-conn1
Connections:
- wire segments 30 -> 35
- no-connect marks 12 -> 11
Changed lines of the file:
@@
 $EndDescr
 $Comp
-L switches1:SW_Push SW1
+L leddings-rescue:SW_Push-switches1 SW1
 U 1 1 5B19308C
 P 3700 3850
 F 0 "SW1" H 3750 3950 50  0000 L CNN
 F 1 "SW_RESET" H 3700 3790 50  0000 C CNN
-F 2 "Buttons_Switches_THT:SW_Tactile_Straight_KSA0Axx1LFTR" H 3700 4050 50  0001 C CNN
+F 2 "Button_Switch_SMD:SW_SPST_B3S-1000" H 3700 4050 50  0001 C CNN
 F 3 "" H 3700 4050 50  0001 C CNN
 	1    3700 3850
@@
 $EndComp
 $Comp
-L device1:R R7
+L leddings-rescue:R-device1 R7
 U 1 1 5B193093
 P 4050 3550
@@
 	0    1    1    0
 $EndComp
-Wire Wire Line
-	3300 3850 3400 3850
 $Comp
 L power1:VCC #PWR019
@@
 $EndComp
 Wire Wire Line
-	4250 4050 3400 4050
-Wire Wire Line
-	3400 4050 3400 3850
-Connection ~ 3400 3850
-$Comp
-L conn1:GS3 SW2
+	4250 4050 4050 4050
+$Comp
+L leddings-rescue:GS3-conn1 SW2
 U 1 1 5B1930B8
 P 7500 4250
@@
 $EndComp
 $Comp
-L device1:R R8
+L leddings-rescue:R-device1 R8
 U 1 1 5B1930D4
 P 6750 3900
@@
 NoConn ~ 6050 4150
 NoConn ~ 6050 4350
-NoConn ~ 6050 4450
 Wire Wire Line
 	6900 4250 6900 2850
@@
 	4150 4450 4250 4450
 Wire Wire Line
-	4050 3850 4250 3850
-Wire Wire Line
-	3400 3850 3500 3850
-Wire Wire Line
 	6750 4250 6900 4250
 Wire Wire Line
@@
 $EndComp
 Wire Wire Line
-	4250 4550 2700 4550
+	4250 4550 4000 4550
 Wire Wire Line
 	2700 4550 2700 3150
@@
 $EndComp
 Wire Wire Line
-	6050 4550 6200 4550
+	6050 4550 6150 4550
+Wire Wire Line
+	6050 4450 6150 4450
+Wire Wire Line
+	6150 4450 6150 4550
+Connection ~ 6150 4550
+Wire Wire Line
+	6150 4550 6200 4550
+$Comp
+L Device:C C6
+U 1 1 5BF8013F
+P 4000 4800
+F 0 "C6" H 4115 4846 50  0000 L CNN
+F 1 "10uF" H 4115 4755 50  0000 L CNN
+F 2 "" H 4038 4650 50  0001 C CNN
+F 3 "~" H 4000 4800 50  0001 C CNN
+	1    4000 4800
+	1    0    0    -1
+$EndComp
+$Comp
+L power:GND #PWR0104
+U 1 1 5BF801ED
+P 4000 5050
+F 0 "#PWR0104" H 4000 4800 50  0001 C CNN
+F 1 "GND" H 4005 4877 50  0000 C CNN
+F 2 "" H 4000 5050 50  0001 C CNN
+F 3 "" H 4000 5050 50  0001 C CNN
+	1    4000 5050
+	1    0    0    -1
+$EndComp
+Wire Wire Line
+	4000 4650 4000 4550
+Connection ~ 4000 4550
+Wire Wire Line
+	4000 4550 2700 4550
+Wire Wire Line
+	4000 5050 4000 4950
+Wire Wire Line
+	3300 3850 3500 3850
+Wire Wire Line
+	4050 4050 4050 3850
+Wire Wire Line
+	4050 3850 4250 3850
 $EndSCHEMATC
