File: uart.sch (KiCad schematic (older format))
At the start: 5 parts

Commit message: added stuff
Parts:
- C3, C4: renamed from C?; footprint (none) -> Capacitors_SMD:C_0805_HandSoldering
- J3: renamed from J?; footprint (none) -> Connectors_USB:USB_Micro-B_Molex-105017-0001
- U2: renamed from U?; footprint (none) -> Housings_SOIC:HTSOP-8-1EP_3.9x4.9mm_Pitch1.27mm
- Y1: renamed from Y?; footprint (none) -> Crystals:Crystal_HC35-U
Changed lines of the file:
@@
 $EndDescr
 $Comp
-L CH340G U?
+L CH340G U2
 U 1 1 5B191996
 P 6750 3650
-F 0 "U?" H 6775 4125 60  0000 C CNN
+F 0 "U2" H 6775 4125 60  0000 C CNN
 F 1 "CH340G" H 6750 3175 60  0000 C CNN
-F 2 "" H 6850 3450 60  0000 C CNN
+F 2 "Housings_SOIC:HTSOP-8-1EP_3.9x4.9mm_Pitch1.27mm" H 6850 3450 60  0001 C CNN
 F 3 "" H 6850 3450 60  0000 C CNN
 	1    6750 3650
@@
 $EndComp
 $Comp
-L USB_A J?
+L USB_A J3
 U 1 1 5B19199D
 P 4250 3700
-F 0 "J?" H 4050 4150 50  0000 L CNN
+F 0 "J3" H 4050 4150 50  0000 L CNN
 F 1 "Micro USB" H 4050 4050 50  0000 L CNN
-F 2 "" H 4400 3650 50  0001 C CNN
+F 2 "Connectors_USB:USB_Micro-B_Molex-105017-0001" H 4400 3650 50  0001 C CNN
 F 3 "" H 4400 3650 50  0001 C CNN
 	1    4250 3700
@@
 	4550 3800 6300 3800
 $Comp
-L VBUS #PWR017
+L VBUS #PWR011
 U 1 1 5B1919A6
 P 4650 3500
-F 0 "#PWR017" H 4650 3350 50  0001 C CNN
+F 0 "#PWR011" H 4650 3350 50  0001 C CNN
 F 1 "VBUS" H 4650 3650 50  0000 C CNN
 F 2 "" H 4650 3500 50  0001 C CNN
@@
 	4550 3500 4650 3500
 $Comp
-L GND #PWR018
+L GND #PWR012
 U 1 1 5B1919AE
 P 4250 4200
-F 0 "#PWR018" H 4250 3950 50  0001 C CNN
+F 0 "#PWR012" H 4250 3950 50  0001 C CNN
 F 1 "GND" H 4250 4050 50  0000 C CNN
 F 2 "" H 4250 4200 50  0001 C CNN
@@
 $EndComp
 $Comp
-L GND #PWR019
+L GND #PWR013
 U 1 1 5B1919B4
 P 6150 3300
-F 0 "#PWR019" H 6150 3050 50  0001 C CNN
+F 0 "#PWR013" H 6150 3050 50  0001 C CNN
 F 1 "GND" H 6150 3150 50  0000 C CNN
 F 2 "" H 6150 3300 50  0001 C CNN
@@
 	4250 4200 4250 4100
 $Comp
-L Crystal Y?
+L Crystal Y1
 U 1 1 5B1919D2
 P 5450 4400
-F 0 "Y?" H 5450 4550 50  0000 C CNN
+F 0 "Y1" H 5450 4550 50  0000 C CNN
 F 1 "12 Mhz Crystal" H 5450 4650 50  0000 C CNN
-F 2 "" H 5450 4400 50  0001 C CNN
+F 2 "Crystals:Crystal_HC35-U" H 5450 4400 50  0001 C CNN
 F 3 "" H 5450 4400 50  0001 C CNN
 	1    5450 4400
@@
 $EndComp
 $Comp
-L C C?
+L C C4
 U 1 1 5B1919D9
 P 5850 4600
-F 0 "C?" H 5875 4700 50  0000 L CNN
+F 0 "C4" H 5875 4700 50  0000 L CNN
 F 1 "22pF" H 5875 4500 50  0000 L CNN
-F 2 "" H 5888 4450 50  0001 C CNN
+F 2 "Capacitors_SMD:C_0805_HandSoldering" H 5888 4450 50  0001 C CNN
 F 3 "" H 5850 4600 50  0001 C CNN
 	1    5850 4600
@@
 $EndComp
 $Comp
-L C C?
+L C C3
 U 1 1 5B1919E0
 P 5050 4600
-F 0 "C?" H 5075 4700 50  0000 L CNN
+F 0 "C3" H 5075 4700 50  0000 L CNN
 F 1 "22pF" H 5075 4500 50  0000 L CNN
-F 2 "" H 5088 4450 50  0001 C CNN
+F 2 "Capacitors_SMD:C_0805_HandSoldering" H 5088 4450 50  0001 C CNN
 F 3 "" H 5050 4600 50  0001 C CNN
 	1    5050 4600
@@
 	5850 4000 5850 4450
 $Comp
-L GND #PWR020
+L GND #PWR014
 U 1 1 5B1919EB
 P 5850 4900
-F 0 "#PWR020" H 5850 4650 50  0001 C CNN
+F 0 "#PWR014" H 5850 4650 50  0001 C CNN
 F 1 "GND" H 5850 4750 50  0000 C CNN
 F 2 "" H 5850 4900 50  0001 C CNN
@@
 $EndComp
 $Comp
-L GND #PWR021
+L GND #PWR015
 U 1 1 5B1919F1
 P 5050 4900
-F 0 "#PWR021" H 5050 4650 50  0001 C CNN
+F 0 "#PWR015" H 5050 4650 50  0001 C CNN
 F 1 "GND" H 5050 4750 50  0000 C CNN
 F 2 "" H 5050 4900 50  0001 C CNN
@@
 NoConn ~ 7200 4000
 $Comp
-L VCC #PWR022
+L VCC #PWR016
 U 1 1 5B191D8F
 P 7350 3200
-F 0 "#PWR022" H 7350 3050 50  0001 C CNN
+F 0 "#PWR016" H 7350 3050 50  0001 C CNN
 F 1 "VCC" H 7350 3350 50  0000 C CNN
 F 2 "" H 7350 3200 50  0001 C CNN
@@
 	7350 3300 7350 3200
 $Comp
-L VCC #PWR023
+L VCC #PWR017
 U 1 1 5B191DCB
 P 6150 3600
-F 0 "#PWR023" H 6150 3450 50  0001 C CNN
+F 0 "#PWR017" H 6150 3450 50  0001 C CNN
 F 1 "VCC" H 6150 3750 50  0000 C CNN
 F 2 "" H 6150 3600 50  0001 C CNN

Commit message: Did a stuff
Parts:
- C3, C4: symbol C -> device1:C
- J5: renamed from J3; symbol USB_A -> conn1:USB_A
- U2: footprint Housings_SOIC:HTSOP-8-1EP_3.9x4.9mm_Pitch1.27mm -> Housings_SOIC:SOIC-16_3.9x9.9mm_Pitch1.27mm; symbol CH340G -> leddings-rescue:CH340G
- Y1: footprint Crystals:Crystal_HC35-U -> Crystals:Crystal_HC49-U_Vertical; symbol Crystal -> device1:Crystal
Connections:
- wire segments 26 -> 29
Changed lines of the file:
@@
-EESchema Schematic File Version 2
-LIBS:power
-LIBS:device
-LIBS:switches
-LIBS:relays
-LIBS:motors
-LIBS:transistors
-LIBS:conn
-LIBS:linear
-LIBS:regul
-LIBS:74xx
-LIBS:cmos4000
-LIBS:adc-dac
-LIBS:memory
-LIBS:xilinx
-LIBS:microcontrollers
-LIBS:dsp
-LIBS:microchip
-LIBS:analog_switches
-LIBS:motorola
-LIBS:texas
-LIBS:intel
-LIBS:audio
-LIBS:interface
-LIBS:digital-audio
-LIBS:philips
-LIBS:display
-LIBS:cypress
-LIBS:siliconi
-LIBS:opto
-LIBS:atmel
-LIBS:contrib
-LIBS:valves
-LIBS:ESP8266
-LIBS:74xgxx
-LIBS:ac-dc
-LIBS:actel
-LIBS:allegro
-LIBS:Altera
-LIBS:analog_devices
-LIBS:battery_management
-LIBS:bbd
-LIBS:bosch
-LIBS:brooktre
-LIBS:cmos_ieee
-LIBS:dc-dc
-LIBS:diode
-LIBS:elec-unifil
-LIBS:ESD_Protection
-LIBS:ftdi
-LIBS:gennum
-LIBS:graphic_symbols
-LIBS:hc11
-LIBS:infineon
-LIBS:intersil
-LIBS:ir
-LIBS:Lattice
-LIBS:leds
-LIBS:LEM
-LIBS:logic_programmable
-LIBS:maxim
-LIBS:mechanical
-LIBS:microchip_dspic33dsc
-LIBS:microchip_pic10mcu
-LIBS:microchip_pic12mcu
-LIBS:microchip_pic16mcu
-LIBS:microchip_pic18mcu
-LIBS:microchip_pic24mcu
-LIBS:microchip_pic32mcu
-LIBS:modules
-LIBS:motor_drivers
-LIBS:msp430
-LIBS:nordicsemi
-LIBS:nxp
-LIBS:nxp_armmcu
-LIBS:onsemi
-LIBS:Oscillators
-LIBS:powerint
-LIBS:Power_Management
-LIBS:pspice
-LIBS:references
-LIBS:rfcom
-LIBS:RFSolutions
-LIBS:sensors
-LIBS:silabs
-LIBS:stm8
-LIBS:stm32
-LIBS:supertex
-LIBS:transf
-LIBS:triac_thyristor
-LIBS:ttl_ieee
-LIBS:video
-LIBS:wiznet
-LIBS:Worldsemi
-LIBS:Xicor
-LIBS:zetex
-LIBS:Zilog
-LIBS:ch34x
+EESchema Schematic File Version 4
 LIBS:leddings-cache
-EELAYER 25 0
+EELAYER 26 0
 EELAYER END
 $Descr A4 11693 8268
@@
 $EndDescr
 $Comp
-L CH340G U2
+L leddings-rescue:CH340G U2
 U 1 1 5B191996
 P 6750 3650
+AR Path="/5B191996" Ref="U2"  Part="1"
+AR Path="/5B191627/5B191996" Ref="U2"  Part="1"
 F 0 "U2" H 6775 4125 60  0000 C CNN
 F 1 "CH340G" H 6750 3175 60  0000 C CNN
-F 2 "Housings_SOIC:HTSOP-8-1EP_3.9x4.9mm_Pitch1.27mm" H 6850 3450 60  0001 C CNN
+F 2 "Housings_SOIC:SOIC-16_3.9x9.9mm_Pitch1.27mm" H 6850 3450 60  0001 C CNN
 F 3 "" H 6850 3450 60  0000 C CNN
 	1    6750 3650
@@
 $EndComp
 $Comp
-L USB_A J3
+L conn1:USB_A J5
 U 1 1 5B19199D
 P 4250 3700
-F 0 "J3" H 4050 4150 50  0000 L CNN
+F 0 "J5" H 4050 4150 50  0000 L CNN
 F 1 "Micro USB" H 4050 4050 50  0000 L CNN
 F 2 "Connectors_USB:USB_Micro-B_Molex-105017-0001" H 4400 3650 50  0001 C CNN
@@
 	4550 3800 6300 3800
 $Comp
-L VBUS #PWR011
+L power1:VBUS #PWR011
 U 1 1 5B1919A6
 P 4650 3500
@@
 	4550 3500 4650 3500
 $Comp
-L GND #PWR012
+L power1:GND #PWR012
 U 1 1 5B1919AE
 P 4250 4200
@@
 $EndComp
 $Comp
-L GND #PWR013
+L power1:GND #PWR013
 U 1 1 5B1919B4
 P 6150 3300
@@
 	6150 3300 6300 3300
 Wire Wire Line
-	4250 4200 4250 4100
-$Comp
-L Crystal Y1
+	4250 4200 4250 4150
+$Comp
+L device1:Crystal Y1
 U 1 1 5B1919D2
 P 5450 4400
 F 0 "Y1" H 5450 4550 50  0000 C CNN
 F 1 "12 Mhz Crystal" H 5450 4650 50  0000 C CNN
-F 2 "Crystals:Crystal_HC35-U" H 5450 4400 50  0001 C CNN
+F 2 "Crystals:Crystal_HC49-U_Vertical" H 5450 4400 50  0001 C CNN
 F 3 "" H 5450 4400 50  0001 C CNN
 	1    5450 4400
@@
 $EndComp
 $Comp
-L C C4
+L device1:C C4
 U 1 1 5B1919D9
 P 5850 4600
@@
 $EndComp
 $Comp
-L C C3
+L device1:C C3
 U 1 1 5B1919E0
 P 5050 4600
@@
 	5300 4400 5050 4400
 Wire Wire Line
-	5050 3900 5050 4450
+	5050 3900 5050 4400
 Wire Wire Line
 	5600 4400 5850 4400
 Wire Wire Line
-	5850 4000 5850 4450
-$Comp
-L GND #PWR014
+	5850 4000 5850 4400
+$Comp
+L power1:GND #PWR014
 U 1 1 5B1919EB
 P 5850 4900
@@
 $EndComp
 $Comp
-L GND #PWR015
+L power1:GND #PWR015
 U 1 1 5B1919F1
 P 5050 4900
@@
 NoConn ~ 7200 4000
 $Comp
-L VCC #PWR016
+L power1:VCC #PWR016
 U 1 1 5B191D8F
 P 7350 3200
@@
 	7350 3300 7350 3200
 $Comp
-L VCC #PWR017
+L power1:VCC #PWR017
 U 1 1 5B191DCB
 P 6150 3600
@@
 	4150 4150 4150 4100
 Connection ~ 4250 4150
+Wire Wire Line
+	5050 4400 5050 4450
+Wire Wire Line
+	5850 4400 5850 4450
+Wire Wire Line
+	4250 4150 4250 4100
 $EndSCHEMATC

Commit message: added pin headers for uart, added power-on-led, improved routing
Parts:
- added J7: Conn_01x04, Pin_Headers:Pin_Header_Straight_1x04_Pitch2.54mm, symbol Connector_Generic:Conn_01x04
Connections:
- wire segments 29 -> 41
Changed lines of the file:
@@
 encoding utf-8
 Sheet 4 5
-Title ""
-Date ""
-Rev ""
+Title "LED Driver"
+Date "2018-10-02"
+Rev "1.0"
 Comp ""
 Comment1 ""
@@
 Wire Wire Line
 	5800 3500 6300 3500
-Text HLabel 7350 3600 2    60   Input ~ 0
+Text HLabel 8500 3600 2    60   Input ~ 0
 DTR
-Text HLabel 7350 3500 2    60   Input ~ 0
+Text HLabel 8500 3500 2    60   Input ~ 0
 RTS
 Wire Wire Line
-	7200 3500 7350 3500
-Wire Wire Line
-	7350 3600 7200 3600
+	7200 3500 7450 3500
+Wire Wire Line
+	8500 3600 7550 3600
 NoConn ~ 7200 3400
 NoConn ~ 7200 3700
@@
 L power1:VCC #PWR016
 U 1 1 5B191D8F
-P 7350 3200
-F 0 "#PWR016" H 7350 3050 50  0001 C CNN
-F 1 "VCC" H 7350 3350 50  0000 C CNN
-F 2 "" H 7350 3200 50  0001 C CNN
-F 3 "" H 7350 3200 50  0001 C CNN
-	1    7350 3200
-	1    0    0    -1
-$EndComp
-Wire Wire Line
-	7200 3300 7350 3300
-Wire Wire Line
-	7350 3300 7350 3200
+P 8400 3200
+F 0 "#PWR016" H 8400 3050 50  0001 C CNN
+F 1 "VCC" H 8400 3350 50  0000 C CNN
+F 2 "" H 8400 3200 50  0001 C CNN
+F 3 "" H 8400 3200 50  0001 C CNN
+	1    8400 3200
+	1    0    0    -1
+$EndComp
+Wire Wire Line
+	7200 3300 8400 3300
+Wire Wire Line
+	8400 3300 8400 3200
 $Comp
 L power1:VCC #PWR017
@@
 Wire Wire Line
 	4250 4150 4250 4100
+$Comp
+L Connector_Generic:Conn_01x04 J7
+U 1 1 5BB37DE2
+P 6700 2300
+F 0 "J7" V 6666 2012 50  0000 R CNN
+F 1 "Conn_01x04" V 6575 2012 50  0000 R CNN
+F 2 "Pin_Headers:Pin_Header_Straight_1x04_Pitch2.54mm" H 6700 2300 50  0001 C CNN
+F 3 "~" H 6700 2300 50  0001 C CNN
+	1    6700 2300
+	0    -1   -1   0
+$EndComp
+Wire Wire Line
+	5800 3100 6700 3100
+Wire Wire Line
+	6700 3100 6700 2500
+Connection ~ 5800 3100
+Wire Wire Line
+	5900 3000 6600 3000
+Wire Wire Line
+	6600 3000 6600 2500
+Connection ~ 5900 3000
+Wire Wire Line
+	6800 2500 6800 3000
+Wire Wire Line
+	6800 3000 7450 3000
+Wire Wire Line
+	7450 3000 7450 3500
+Connection ~ 7450 3500
+Wire Wire Line
+	7450 3500 8500 3500
+Wire Wire Line
+	7550 3600 7550 2900
+Wire Wire Line
+	7550 2900 6900 2900
+Wire Wire Line
+	6900 2900 6900 2500
+Connection ~ 7550 3600
+Wire Wire Line
+	7550 3600 7200 3600
 $EndSCHEMATC

Commit message: changed some parts to smd, fixed some design errors
Parts:
- added C5: 10uF, Capacitor_SMD:C_0805_2012Metric_Pad1.15x1.40mm_HandSolder, symbol Device:C
- C3, C4: symbol device1:C -> leddings-rescue:C-device1
- J5: symbol conn1:USB_A -> leddings-rescue:USB_A-conn1
- Y1: symbol device1:Crystal -> leddings-rescue:Crystal-device1
Connections:
- wire segments 41 -> 44
Changed lines of the file:
@@
 $EndComp
 $Comp
-L conn1:USB_A J5
+L leddings-rescue:USB_A-conn1 J5
 U 1 1 5B19199D
 P 4250 3700
@@
 F 3 "" H 6150 3300 50  0001 C CNN
 	1    6150 3300
-	0    1    1    0
+	-1   0    0    1
 $EndComp
 Wire Wire Line
@@
 	4250 4200 4250 4150
 $Comp
-L device1:Crystal Y1
+L leddings-rescue:Crystal-device1 Y1
 U 1 1 5B1919D2
 P 5450 4400
@@
 $EndComp
 $Comp
-L device1:C C4
+L leddings-rescue:C-device1 C4
 U 1 1 5B1919D9
 P 5850 4600
@@
 $EndComp
 $Comp
-L device1:C C3
+L leddings-rescue:C-device1 C3
 U 1 1 5B1919E0
 P 5050 4600
@@
 L power1:VCC #PWR016
 U 1 1 5B191D8F
-P 8400 3200
-F 0 "#PWR016" H 8400 3050 50  0001 C CNN
-F 1 "VCC" H 8400 3350 50  0000 C CNN
-F 2 "" H 8400 3200 50  0001 C CNN
-F 3 "" H 8400 3200 50  0001 C CNN
-	1    8400 3200
-	1    0    0    -1
-$EndComp
-Wire Wire Line
-	7200 3300 8400 3300
-Wire Wire Line
-	8400 3300 8400 3200
-$Comp
-L power1:VCC #PWR017
-U 1 1 5B191DCB
-P 6150 3600
-F 0 "#PWR017" H 6150 3450 50  0001 C CNN
-F 1 "VCC" H 6150 3750 50  0000 C CNN
-F 2 "" H 6150 3600 50  0001 C CNN
-F 3 "" H 6150 3600 50  0001 C CNN
-	1    6150 3600
-	0    -1   -1   0
-$EndComp
-Wire Wire Line
-	6150 3600 6300 3600
+P 8700 3150
+F 0 "#PWR016" H 8700 3000 50  0001 C CNN
+F 1 "VCC" H 8700 3300 50  0000 C CNN
+F 2 "" H 8700 3150 50  0001 C CNN
+F 3 "" H 8700 3150 50  0001 C CNN
+	1    8700 3150
+	1    0    0    -1
+$EndComp
+Wire Wire Line
+	7200 3300 7800 3300
+Wire Wire Line
+	8700 3300 8700 3150
 Wire Wire Line
 	4250 4150 4150 4150
@@
 Wire Wire Line
 	7550 3600 7200 3600
+$Comp
+L Device:C C5
+U 1 1 5BF740A2
+P 7800 3100
+F 0 "C5" H 7915 3146 50  0000 L CNN
+F 1 "10uF" H 7915 3055 50  0000 L CNN
+F 2 "Capacitor_SMD:C_0805_2012Metric_Pad1.15x1.40mm_HandSolder" H 7838 2950 50  0001 C CNN
+F 3 "~" H 7800 3100 50  0001 C CNN
+	1    7800 3100
+	1    0    0    -1
+$EndComp
+Wire Wire Line
+	5850 3600 6300 3600
+$Comp
+L power:GND #PWR0102
+U 1 1 5BF77837
+P 7800 2850
+F 0 "#PWR0102" H 7800 2600 50  0001 C CNN
+F 1 "GND" H 7805 2677 50  0000 C CNN
+F 2 "" H 7800 2850 50  0001 C CNN
+F 3 "" H 7800 2850 50  0001 C CNN
+	1    7800 2850
+	-1   0    0    1
+$EndComp
+Wire Wire Line
+	7800 3250 7800 3300
+Connection ~ 7800 3300
+$Comp
+L power:VCC #PWR0103
+U 1 1 5BF7D5D8
+P 5850 3600
+F 0 "#PWR0103" H 5850 3450 50  0001 C CNN
+F 1 "VCC" V 5868 3727 50  0000 L CNN
+F 2 "" H 5850 3600 50  0001 C CNN
+F 3 "" H 5850 3600 50  0001 C CNN
+	1    5850 3600
+	0    -1   -1   0
+$EndComp
+Wire Wire Line
+	7800 3300 8700 3300
+Wire Wire Line
+	7800 2850 7800 2950
 $EndSCHEMATC
